Commit message: fix urdf path

File: src/mower_robot_description/urdf/mower_robot.urdf (robot description, URDF)
Before this commit: robot mower_robot, 8 links, 7 joints
Links:
- link back_camera_link_1: geometry collision mesh filename=package://mower_robot_description/meshes/back_camera_link_1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 scale=0.001 0.001 0.001; visual mesh filename=package://mower_robot_description/meshes/back_camera_link_1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 scale=0.001 0.001 0.001
- link base_link: geometry collision mesh filename=package://mower_robot_description/meshes/base_link.stl scale=0.001 0.001 0.001; visual mesh filename=package://mower_robot_description/meshes/base_link.stl scale=0.001 0.001 0.001
- link caster_wheel_link_1: geometry collision mesh filename=package://mower_robot_description/meshes/caster_wheel_link_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 scale=0.001 0.001 0.001; visual mesh filename=package://mower_robot_description/meshes/caster_wheel_link_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 scale=0.001 0.001 0.001
- link caster_yaw_link_1: geometry collision mesh filename=package://mower_robot_description/meshes/caster_yaw_link_1.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 scale=0.001 0.001 0.001; visual mesh filename=../meshes/caster_yaw_link_1.stl scale=0.001 0.001 0.001
- link depth_camera_link_1: geometry collision mesh filename=package://mower_robot_description/meshes/depth_camera_link_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 scale=0.001 0.001 0.001; visual mesh filename=package://mower_robot_description/meshes/depth_camera_link_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 scale=0.001 0.001 0.001
- link imu_link_1: geometry collision mesh filename=package://mower_robot_description/meshes/imu_link_1.stl scale=0.001 0.001 0.001; visual mesh filename=package://mower_robot_description/meshes/imu_link_1.stl scale=0.001 0.001 0.001
- link left_wheel_link_1: geometry collision mesh filename=package://mower_robot_description/meshes/left_wheel_link_1.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 scale=0.001 0.001 0.001; visual mesh filename=package://mower_robot_description/meshes/left_wheel_link_1.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 scale=0.001 0.001 0.001
- link left_wheel_link_2: geometry collision mesh filename=package://mower_robot_description/meshes/left_wheel_link_2.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 scale=0.001 0.001 0.001; visual mesh filename=package://mower_robot_description/meshes/left_wheel_link_2.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 scale=0.001 0.001 0.001

Commit message: update mower robot urdf

File: src/mower_robot_description/urdf/mower_robot.urdf (robot description, URDF)
Before this commit: robot mower_robot, 8 links, 7 joints
Links:
- link caster_yaw_link_1: geometry collision mesh filename=package://mower_robot_description/meshes/caster_yaw_link_1.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 scale=0.001 0.001 0.001; visual mesh filename=package://mower_robot_description/meshes/caster_yaw_link_1.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 scale=0.001 0.001 0.001

File: src/mower_robot_description/urdf/mower_robot.xacro (robot description, xacro)
@@ -14,5 +14,5 @@
     <origin xyz="0 0 0" rpy="0 0 0"/>
     <geometry>
-      <mesh filename="file://$(find mower_robot_description)/meshes/base_link.stl" scale="0.001 0.001 0.001"/>
+      <mesh filename="package://mower_robot_description/meshes/base_link.stl" scale="0.001 0.001 0.001"/>
     </geometry>
     <material name="silver"/>
@@ -21,5 +21,5 @@
     <origin xyz="0 0 0" rpy="0 0 0"/>
     <geometry>
-      <mesh filename="file://$(find mower_robot_description)/meshes/base_link.stl" scale="0.001 0.001 0.001"/>
+      <mesh filename="package://mower_robot_description/meshes/base_link.stl" scale="0.001 0.001 0.001"/>
     </geometry>
   </collision>
@@ -34,5 +34,5 @@
     <origin xyz="-0.01938 0.190279 0.1125" rpy="0 0 0"/>
     <geometry>
-      <mesh filename="file://$(find mower_robot_description)/meshes/caster_wheel_link_1.stl" scale="0.001 0.001 0.001"/>
+      <mesh filename="package://mower_robot_description/meshes/caster_wheel_link_1.stl" scale="0.001 0.001 0.001"/>
     </geometry>
     <material name="silver"/>
@@ -41,5 +41,5 @@
     <origin xyz="-0.01938 0.190279 0.1125" rpy="0 0 0"/>
     <geometry>
-      <mesh filename="file://$(find mower_robot_description)/meshes/caster_wheel_link_1.stl" scale="0.001 0.001 0.001"/>
+      <mesh filename="package://mower_robot_description/meshes/caster_wheel_link_1.stl" scale="0.001 0.001 0.001"/>
     </geometry>
   </collision>
@@ -54,5 +54,5 @@
     <origin xyz="0.0 0.1665 0.043" rpy="0 0 0"/>
     <geometry>
-      <mesh filename="file://$(find mower_robot_description)/meshes/caster_yaw_link_1.stl" scale="0.001 0.001 0.001"/>
+      <mesh filename="package://mower_robot_description/meshes/caster_yaw_link_1.stl" scale="0.001 0.001 0.001"/>
     </geometry>
     <material name="silver"/>
@@ -61,5 +61,5 @@
     <origin xyz="0.0 0.1665 0.043" rpy="0 0 0"/>
     <geometry>
-      <mesh filename="file://$(find mower_robot_description)/meshes/caster_yaw_link_1.stl" scale="0.001 0.001 0.001"/>
+      <mesh filename="package://mower_robot_description/meshes/caster_yaw_link_1.stl" scale="0.001 0.001 0.001"/>
     </geometry>
   </collision>
@@ -74,5 +74,5 @@
     <origin xyz="-0.12 -0.15 0.06" rpy="0 0 0"/>
     <geometry>
-      <mesh filename="file://$(find mower_robot_description)/meshes/left_wheel_link_1.stl" scale="0.001 0.001 0.001"/>
+      <mesh filename="package://mower_robot_description/meshes/left_wheel_link_1.stl" scale="0.001 0.001 0.001"/>
     </geometry>
     <material name="silver"/>
@@ -81,5 +81,5 @@
     <origin xyz="-0.12 -0.15 0.06" rpy="0 0 0"/>
     <geometry>
-      <mesh filename="file://$(find mower_robot_description)/meshes/left_wheel_link_1.stl" scale="0.001 0.001 0.001"/>
+      <mesh filename="package://mower_robot_description/meshes/left_wheel_link_1.stl" scale="0.001 0.001 0.001"/>
     </geometry>
   </collision>
@@ -94,5 +94,5 @@
     <origin xyz="0.12 -0.15 0.06" rpy="0 0 0"/>
     <geometry>
-      <mesh filename="file://$(find mower_robot_description)/meshes/left_wheel_link_2.stl" scale="0.001 0.001 0.001"/>
+      <mesh filename="package://mower_robot_description/meshes/left_wheel_link_2.stl" scale="0.001 0.001 0.001"/>
     </geometry>
     <material name="silver"/>
@@ -101,5 +101,5 @@
     <origin xyz="0.12 -0.15 0.06" rpy="0 0 0"/>
     <geometry>
-      <mesh filename="file://$(find mower_robot_description)/meshes/left_wheel_link_2.stl" scale="0.001 0.001 0.001"/>
+      <mesh filename="package://mower_robot_description/meshes/left_wheel_link_2.stl" scale="0.001 0.001 0.001"/>
     </geometry>
   </collision>
@@ -114,5 +114,5 @@
     <origin xyz="0.000633 -0.194 0.07" rpy="0 0 0"/>
     <geometry>
-      <mesh filename="file://$(find mower_robot_description)/meshes/imu_link_1.stl" scale="0.001 0.001 0.001"/>
+      <mesh filename="package://mower_robot_description/meshes/imu_link_1.stl" scale="0.001 0.001 0.001"/>
     </geometry>
     <material name="silver"/>
@@ -121,5 +121,5 @@
     <origin xyz="0.000633 -0.194 0.07" rpy="0 0 0"/>
     <geometry>
-      <mesh filename="file://$(find mower_robot_description)/meshes/imu_link_1.stl" scale="0.001 0.001 0.001"/>
+      <mesh filename="package://mower_robot_description/meshes/imu_link_1.stl" scale="0.001 0.001 0.001"/>
     </geometry>
   </collision>
@@ -134,5 +134,5 @@
     <origin xyz="0.0 -0.2024 0.145" rpy="0 0 0"/>
     <geometry>
-      <mesh filename="file://$(find mower_robot_description)/meshes/back_camera_link_1.stl" scale="0.001 0.001 0.001"/>
+      <mesh filename="package://mower_robot_description/meshes/back_camera_link_1.stl" scale="0.001 0.001 0.001"/>
     </geometry>
     <material name="silver"/>
@@ -141,5 +141,5 @@
     <origin xyz="0.0 -0.2024 0.145" rpy="0 0 0"/>
     <geometry>
-      <mesh filename="file://$(find mower_robot_description)/meshes/back_camera_link_1.stl" scale="0.001 0.001 0.001"/>
+      <mesh filename="package://mower_robot_description/meshes/back_camera_link_1.stl" scale="0.001 0.001 0.001"/>
     </geometry>
   </collision>
@@ -154,5 +154,5 @@
     <origin xyz="-0.0225 0.199445 -0.0175" rpy="0 0 0"/>
     <geometry>
-      <mesh filename="file://$(find mower_robot_description)/meshes/depth_camera_link_1.stl" scale="0.001 0.001 0.001"/>
+      <mesh filename="package://mower_robot_description/meshes/depth_camera_link_1.stl" scale="0.001 0.001 0.001"/>
     </geometry>
     <material name="silver"/>
@@ -161,5 +161,5 @@
     <origin xyz="-0.0225 0.199445 -0.0175" rpy="0 0 0"/>
     <geometry>
-      <mesh filename="file://$(find mower_robot_description)/meshes/depth_camera_link_1.stl" scale="0.001 0.001 0.001"/>
+      <mesh filename="package://mower_robot_description/meshes/depth_camera_link_1.stl" scale="0.001 0.001 0.001"/>
     </geometry>
   </collision>
