Commit message: fix ros2 control & disable diff controller tf publish

File: src/mower_description/mower_robot/real_robot_ros2_control.xacro (robot description, xacro)
@@ -30,9 +30,3 @@
     </joint>
   </ros2_control>
-   <gazebo>
-    <plugin name="gazebo_ros2_control" filename="libgazebo_ros2_control.so">
-      <use_sim_time>true</use_sim_time>
-      <parameters>$(find mower_controller)/controllers/diff_drive_controller.yaml</parameters>
-    </plugin>
-  </gazebo>
 </robot>

File: src/mower_description/mower_robot/robot.gazebo.xacro (robot description, xacro)
@@ -50,4 +50,40 @@
     </plugin>
   </gazebo>
+  <!-- ============================================================ -->
+  <!--  ros2_control Hardware Interface（Gazebo 模擬用）            -->
+  <!--  使用 GazeboSimSystem plugin，讓 gz_ros2_control 與 Gazebo 溝通
+  <!-- ============================================================ -->
+  <ros2_control name="GazeboSystem" type="system">
+    <hardware>
+      <plugin>gz_ros2_control/GazeboSimSystem</plugin>
+    </hardware>
+    <!-- 左輪：velocity command + position/velocity state -->
+    <joint name="left_wheel_joint">
+      <command_interface name="velocity">
+        <param name="min">-6</param>
+        <param name="max">6</param>
+      </command_interface>
+      <state_interface name="position"/>
+      <state_interface name="velocity"/>
+    </joint>
+    <!-- 右輪：velocity command + position/velocity state -->
+    <joint name="right_wheel_joint">
+      <command_interface name="velocity">
+        <param name="min">-6</param>
+        <param name="max">6</param>
+      </command_interface>
+      <state_interface name="position"/>
+      <state_interface name="velocity"/>
+    </joint>
+    <!-- 割草刀盤：effort command + effort state only -->
+    <joint name="mower_joint">
+      <command_interface name="effort">
+        <param name="min">-100</param>
+        <param name="max">100</param>
+      </command_interface>
+      <state_interface name="effort"/>
+      <state_interface name="position"/>
+    </joint>
+  </ros2_control>
   <!-- ============================================================ -->
   <!--  3. IMU Sensor（掛載在 imu_link 上）                         -->

File: src/mower_description/mower_robot/robot.urdf.xacro (robot description, xacro)
@@ -368,38 +368,3 @@
     <limit effort="100" velocity="6"/>
   </joint>
-  <!-- ============================================================ -->
-  <!--  ros2_control Hardware Interface                             -->
-  <!--  使用 GazeboSystem plugin，讓 gz_ros2_control 與 Gazebo 溝通  -->
-  <!-- ============================================================ -->
-  <ros2_control name="GazeboSystem" type="system">
-    <hardware>
-      <plugin>gz_ros2_control/GazeboSimSystem</plugin>
-    </hardware>
-    <!-- 左輪：velocity command + position/velocity state -->
-    <joint name="left_wheel_joint">
-      <command_interface name="velocity">
-        <param name="min">-6</param>
-        <param name="max">6</param>
-      </command_interface>
-      <state_interface name="position"/>
-      <state_interface name="velocity"/>
-    </joint>
-    <!-- 右輪：velocity command + position/velocity state -->
-    <joint name="right_wheel_joint">
-      <command_interface name="velocity">
-        <param name="min">-6</param>
-        <param name="max">6</param>
-      </command_interface>
-      <state_interface name="position"/>
-      <state_interface name="velocity"/>
-    </joint>
-    <!-- 割草刀盤：effort command + effort state only -->
-    <joint name="mower_joint">
-      <command_interface name="effort">
-        <param name="min">-100</param>
-        <param name="max">100</param>
-      </command_interface>
-      <state_interface name="effort"/>
-    </joint>
-  </ros2_control>
 </robot>

Commit message: Fix mower motor controller

File: src/mower_description/mower_robot/real_robot_ros2_control.xacro (robot description, xacro)
@@ -29,4 +29,14 @@
       <state_interface name="velocity"/>
     </joint>
+    <!-- Mower Blade Joint (for mower_blade_controller / JointGroupEffortController) -->
+    <joint name="mower_joint">
+      <command_interface name="effort">
+        <param name="min">-100</param>
+        <param name="max">100</param>
+      </command_interface>
+      <state_interface name="position"/>
+      <state_interface name="velocity"/>
+      <state_interface name="effort"/>
+    </joint>
   </ros2_control>
 </robot>
