Commit message: Add mower_blade_controller

File: src/mower_description/mower_robot/robot.urdf.xacro (robot description, xacro)
@@ -360,10 +360,11 @@
   </joint>
   <!-- Joint: base_link → connector -->
-  <joint name="mower_joint" type="revolute">
+  <!-- continuous: 刀盤需要無限旋轉，不能用 revolute（有 -π~π 限制） -->
+  <joint name="mower_joint" type="continuous">
     <origin xyz="0.0145303 0.0155339 -0.0549528" rpy="0 -0 3.14159"/>
     <parent link="base_link"/>
     <child link="connector"/>
     <axis xyz="0 0 1"/>
-    <limit effort="10" velocity="6" lower="-3.14159" upper="3.14159"/>
+    <limit effort="100" velocity="6"/>
   </joint>
   <!-- ============================================================ -->
@@ -393,4 +394,12 @@
       <state_interface name="velocity"/>
     </joint>
+    <!-- 割草刀盤：effort command + effort state only -->
+    <joint name="mower_joint">
+      <command_interface name="effort">
+        <param name="min">-100</param>
+        <param name="max">100</param>
+      </command_interface>
+      <state_interface name="effort"/>
+    </joint>
   </ros2_control>
 </robot>

Commit message: Fix mower base footprint orientation
Rotate the CAD-derived base_link frame relative to base_footprint so the base_footprint X axis points in the mower forward direction.

File: src/mower_description/mower_robot/robot.urdf.xacro (robot description, xacro)
@@ -32,5 +32,6 @@
   <link name="base_footprint"/>
   <joint name="base_footprint_joint" type="fixed">
-    <origin xyz="0 0 0" rpy="0 0 0"/>
+    <!-- Rotate CAD frame so base_footprint +X is the mower forward direction. -->
+    <origin xyz="0 0 0" rpy="0 0 1.5708"/>
     <parent link="base_footprint"/>
     <child link="base_link"/>
