Commit message: refactor(sim): replace gazebo bridge with ros2_control

File: src/mower_description/mower_robot/robot.gazebo.xacro (robot description, xacro)
@@ -30,39 +30,22 @@
   </gazebo>
   <!-- ============================================================ -->
-  <!--  1. Differential Drive Plugin                                -->
-  <!--     gz-sim-diff-drive-system                                 -->
-  <!--     訂閱: /cmd_vel                                           -->
-  <!--     發布: /odom, /tf                                         -->
+  <!--  1. gz_ros2_control Plugin                                   -->
+  <!--     取代舊的 diff_drive + joint_state_publisher plugins       -->
+  <!--     由 ros2_control 的 diff_drive_controller 負責:            -->
+  <!--       訂閱: /diff_drive_controller/cmd_vel (remapped /cmd_vel)-->
+  <!--       發布: /diff_drive_controller/odom   (remapped /odom)   -->
+  <!--             /tf (odom → base_footprint)                      -->
+  <!--             /joint_states (via joint_state_broadcaster)       -->
   <!-- ============================================================ -->
   <gazebo>
-    <plugin
-      filename="gz-sim-diff-drive-system"
-      name="gz::sim::systems::DiffDrive">
-      <!-- 左右輪 joint 名稱（對應 robot.urdf.xacro 的 joint name）-->
-      <left_joint>left_wheel_joint</left_joint>
-      <right_joint>right_wheel_joint</right_joint>
-      <!-- 車輪規格（單位: 公尺）-->
-      <wheel_separation>0.23600</wheel_separation>  <!-- 左右輪距 -->
-      <wheel_radius>0.05100</wheel_radius>           <!-- 車輪半徑 -->
-      <!-- Odometry 設定 -->
-      <odom_publish_frequency>50</odom_publish_frequency>
-      <!-- ROS topics -->
-      <topic>/cmd_vel</topic>
-      <odom_topic>/odom</odom_topic>
-      <tf_topic>/tf</tf_topic>
-      <!-- Frame 名稱 -->
-      <frame_id>odom</frame_id>
-      <child_frame_id>base_footprint</child_frame_id>
-    </plugin>
-  </gazebo>
-  <!-- ============================================================ -->
-  <!--  2. Joint State Publisher Plugin                             -->
-  <!--     發布所有 joint 的角度，給 robot_state_publisher 使用     -->
-  <!-- ============================================================ -->
-  <gazebo>
-    <plugin
-      filename="gz-sim-joint-state-publisher-system"
-      name="gz::sim::systems::JointStatePublisher">
-      <topic>/joint_states</topic>
+    <plugin filename="libgz_ros2_control-system.so" name="gz_ros2_control::GazeboSimROS2ControlPlugin">
+      <!-- 指向 controller_manager 參數檔，定義 diff_drive_controller 等 -->
+      <parameters>$(find mower_description)/config/controllers.yaml</parameters>
+      <!-- ↓ 在 controller_manager 層級做 remap（spawner 的 remappings= 無效！
+           因為 controller 是跑在 controller_manager 進程裡，不在 spawner 進程裡）-->
+      <ros>
+        <remapping>/diff_drive_controller/cmd_vel:=/cmd_vel</remapping>
+        <remapping>/diff_drive_controller/odom:=/odom</remapping>
+      </ros>
     </plugin>
   </gazebo>
@@ -176,15 +159,3 @@
     </sensor>
   </gazebo>
-  <!-- ============================================================ -->
-  <!--  5. ROS2 橋接 Plugin (gz_ros2_control 或 ros_gz_bridge)      -->
-  <!--     讓 gz-sim 的 topic 橋接到 ROS2                           -->
-  <!-- ============================================================ -->
-  <gazebo>
-    <plugin
-      filename="gz-sim-ros2-control-system"
-      name="gz_ros2_control::GazeboSimROS2ControlPlugin">
-      <!-- 如果你使用 ros2_control，在這裡指定 URDF 中的 controller -->
-      <!-- 如果只用 diff_drive plugin，可以刪除此 plugin -->
-    </plugin>
-  </gazebo>
 </robot>

File: src/mower_description/mower_robot/robot.urdf.xacro (robot description, xacro)
@@ -84,9 +84,10 @@
   </link>
   <!-- Joint: base_link → left_wheel_link -->
+  <!-- rpy x=+1.5708: 輪子朝外安裝，Z 軸向內，需用 0 0 -1 讓正速度=前進 -->
   <joint name="left_wheel_joint" type="continuous">
     <origin xyz="0.13253 0.165534 -0.00295275" rpy="1.5708 1.22081 -1.5708"/>
     <parent link="base_link"/>
     <child link="left_wheel_link"/>
-    <axis xyz="0 0 1"/>
+    <axis xyz="0 0 -1"/>
     <limit effort="10" velocity="6"/>
   </joint>
@@ -116,4 +117,5 @@
   </link>
   <!-- Joint: base_link → right_wheel_link -->
+  <!-- rpy x=-1.5708: 輪子朝外安裝（另一側），Z 軸向外，用 0 0 1 讓正速度=前進 -->
   <joint name="right_wheel_joint" type="continuous">
     <origin xyz="-0.10347 0.165534 -0.00295275" rpy="-1.5708 1.51106 -1.5708"/>
@@ -365,3 +367,30 @@
     <limit effort="10" velocity="6" lower="-3.14159" upper="3.14159"/>
   </joint>
+  <!-- ============================================================ -->
+  <!--  ros2_control Hardware Interface                             -->
+  <!--  使用 GazeboSystem plugin，讓 gz_ros2_control 與 Gazebo 溝通  -->
+  <!-- ============================================================ -->
+  <ros2_control name="GazeboSystem" type="system">
+    <hardware>
+      <plugin>gz_ros2_control/GazeboSimSystem</plugin>
+    </hardware>
+    <!-- 左輪：velocity command + position/velocity state -->
+    <joint name="left_wheel_joint">
+      <command_interface name="velocity">
+        <param name="min">-6</param>
+        <param name="max">6</param>
+      </command_interface>
+      <state_interface name="position"/>
+      <state_interface name="velocity"/>
+    </joint>
+    <!-- 右輪：velocity command + position/velocity state -->
+    <joint name="right_wheel_joint">
+      <command_interface name="velocity">
+        <param name="min">-6</param>
+        <param name="max">6</param>
+      </command_interface>
+      <state_interface name="position"/>
+      <state_interface name="velocity"/>
+    </joint>
+  </ros2_control>
 </robot>

Commit message: chore: update Onshape mower model

File: src/mower_description/mower_robot/robot.gazebo.xacro (robot description, xacro)
@@ -28,4 +28,10 @@
     <mu1>0.01</mu1>
     <mu2>0.01</mu2>
+  </gazebo>
+  <gazebo reference="back_camera_link">
+    <material>Gazebo/Black</material>
+  </gazebo>
+  <gazebo reference="depth_camera_link">
+    <material>Gazebo/Black</material>
   </gazebo>
   <!-- ============================================================ -->
@@ -40,4 +46,6 @@
   <gazebo>
     <plugin filename="libgz_ros2_control-system.so" name="gz_ros2_control::GazeboSimROS2ControlPlugin">
+      <robot_param>robot_description</robot_param>
+      <robot_param_node>robot_state_publisher</robot_param_node>
       <!-- 指向 controller_manager 參數檔，定義 diff_drive_controller 等 -->
       <parameters>$(find mower_description)/config/controllers.yaml</parameters>
@@ -45,4 +53,5 @@
            因為 controller 是跑在 controller_manager 進程裡，不在 spawner 進程裡）-->
       <ros>
+        <remapping>~/robot_description:=/robot_description</remapping>
         <remapping>/diff_drive_controller/cmd_vel:=/cmd_vel</remapping>
         <remapping>/diff_drive_controller/odom:=/odom</remapping>
@@ -195,3 +204,91 @@
     </sensor>
   </gazebo>
+  <!-- ============================================================ -->
+  <!--  5. Back Camera Sensor（掛載在 back_camera_link 上）          -->
+  <!--     發布 gz topics: /back_camera/image_raw,                  -->
+  <!--                    /back_camera/camera_info                  -->
+  <!-- ============================================================ -->
+  <gazebo reference="back_camera_link">
+    <sensor name="back_camera_sensor" type="camera">
+      <always_on>true</always_on>
+      <update_rate>15</update_rate>
+      <visualize>true</visualize>
+      <topic>back_camera/image_raw</topic>
+      <gz_frame_id>back_camera_link</gz_frame_id>
+      <camera name="back_camera">
+        <camera_info_topic>back_camera/camera_info</camera_info_topic>
+        <horizontal_fov>1.3962634</horizontal_fov>
+        <image>
+          <width>640</width>
+          <height>480</height>
+          <format>R8G8B8</format>
+        </image>
+        <clip>
+          <near>0.05</near>
+          <far>10.0</far>
+        </clip>
+        <noise>
+          <type>gaussian</type>
+          <mean>0.0</mean>
+          <stddev>0.005</stddev>
+        </noise>
+        <distortion>
+          <k1>0.0</k1>
+          <k2>0.0</k2>
+          <k3>0.0</k3>
+          <p1>0.0</p1>
+          <p2>0.0</p2>
+          <center>0.5 0.5</center>
+        </distortion>
+      </camera>
+    </sensor>
+  </gazebo>
+  <!-- ============================================================ -->
+  <!--  6. Front Depth Camera Sensor（掛載在 depth_camera_link 上）  -->
+  <!--     發布 gz topics: /front_depth_camera/image_raw,           -->
+  <!--                    /front_depth_camera/depth_image,          -->
+  <!--                    /front_depth_camera/camera_info,          -->
+  <!--                    /front_depth_camera/points                -->
+  <!-- ============================================================ -->
+  <gazebo reference="depth_camera_link">
+    <sensor name="front_depth_camera_sensor" type="rgbd_camera">
+      <always_on>true</always_on>
+      <update_rate>15</update_rate>
+      <visualize>true</visualize>
+      <topic>front_depth_camera</topic>
+      <gz_frame_id>depth_camera_link</gz_frame_id>
+      <camera name="front_depth_camera">
+        <camera_info_topic>front_depth_camera/camera_info</camera_info_topic>
+        <horizontal_fov>1.3962634</horizontal_fov>
+        <image>
+          <width>640</width>
+          <height>480</height>
+          <format>R8G8B8</format>
+        </image>
+        <clip>
+          <near>0.08</near>
+          <far>8.0</far>
+        </clip>
+        <depth_camera>
+          <clip>
+            <near>0.08</near>
+            <far>8.0</far>
+          </clip>
+        </depth_camera>
+        <noise>
+          <type>gaussian</type>
+          <mean>0.0</mean>
+          <stddev>0.005</stddev>
+        </noise>
+        <distortion>
+          <k1>0.0</k1>
+          <k2>0.0</k2>
+          <k3>0.0</k3>
+          <p1>0.0</p1>
+          <p2>0.0</p2>
+          <center>0.5 0.5</center>
+        </distortion>
+      </camera>
+    </sensor>
+  </gazebo>
 </robot>

File: src/mower_description/mower_robot/robot.urdf (robot description, URDF)
Before this commit: robot mower_robot, 10 links, 9 joints
Joints:
- joint back_camera_joint: origin xyz=0.0145303 0.218752 0.0620472 rpy=-1.5708 -0 0 -> xyz=-0.206981 0.000572341 0.0620472 rpy=-1.5708 -0 1.5708
- joint caster_wheel_joint: origin xyz=-0.0255 0.0170526 -0.0695 rpy=1.5708 1.52376 -3.14159 -> xyz=-0.0255 0.0170526 -0.0695 rpy=1.5708 0.37367 -3.14159
- joint caster_yaw_joint: limit lower=-3.14159 upper=3.14159 effort=10 velocity=6 -> lower=-6.28319 upper=0 effort=10 velocity=6; origin xyz=0.0145303 -0.150966 0.0155472 rpy=0 -0 -1.5708 -> xyz=0.162737 0.000572341 0.0155472 rpy=-0 0 3.14159
- joint depth_camera_joint: origin xyz=0.0370303 -0.183912 0.0740472 rpy=-1.5708 -0 0 -> xyz=0.195683 0.0230723 0.0740472 rpy=-1.5708 -0 1.5708
- joint imu_joint: origin xyz=0.015897 0.209534 -0.0129528 rpy=3.14159 -0 0 -> xyz=-0.197763 0.00193904 -0.0129528 rpy=3.14159 -0 1.5708
- joint left_wheel_joint: origin xyz=0.13253 0.165534 -0.00295275 rpy=1.5708 1.22081 -1.5708 -> xyz=-0.153763 0.118572 -0.00295275 rpy=1.5708 1.24431 -0
- joint mower_joint: origin xyz=0.0145303 0.0155339 -0.0549528 rpy=0 -0 3.14159 -> xyz=-0.00376282 0.000572341 -0.0549528 rpy=0 -0 -1.5708
- joint pad_joint: origin xyz=-0 0 -0.018 rpy=0 -0 -0 -> xyz=0 0 -0.018 rpy=0 -0 -0
- joint right_wheel_joint: origin xyz=-0.10347 0.165534 -0.00295275 rpy=-1.5708 1.51106 -1.5708 -> xyz=-0.153763 -0.117428 -0.00295275 rpy=-1.5708 1.53456 -0

Commit message: feat: update simulation world and camera setup

File: src/mower_description/mower_robot/robot.gazebo.xacro (robot description, xacro)
@@ -214,6 +214,7 @@
       <update_rate>15</update_rate>
       <visualize>true</visualize>
+      <pose>0 0 0 1.5708 -1.5708 0</pose>
       <topic>back_camera/image_raw</topic>
-      <gz_frame_id>back_camera_link</gz_frame_id>
+      <gz_frame_id>back_camera_rotated_frame</gz_frame_id>
       <camera name="back_camera">
         <camera_info_topic>back_camera/camera_info</camera_info_topic>
@@ -256,4 +257,5 @@
       <update_rate>15</update_rate>
       <visualize>true</visualize>
+      <pose>0 0 0 0 0 0</pose>
       <topic>front_depth_camera</topic>
       <gz_frame_id>depth_camera_link</gz_frame_id>

File: src/mower_description/mower_robot/robot.urdf (robot description, URDF)
Before this commit: robot mower_robot, 10 links, 9 joints
Links:
- added link back_camera_rotated_frame; visual box size=0.7 0.014 0.014; visual box size=0.7 0.014 0.014
Joints:
- added joint back_camera_rotated_joint: type fixed, parent back_camera_link, child back_camera_rotated_frame, origin xyz=0 0 0 rpy=0 0 1.5708

File: src/mower_description/mower_robot/robot.urdf.xacro (robot description, xacro)
@@ -26,4 +26,7 @@
   <material name="silver_material">
     <color rgba="0.6 0.6 0.6 1"/>
+  </material>
+  <material name="camera_direction_material">
+    <color rgba="0 0.85 1 0.75"/>
   </material>
   <!-- ============================================================ -->
@@ -250,4 +253,53 @@
     <child link="back_camera_link"/>
   </joint>
+  <link name="back_camera_rotated_frame">
+    <visual name="back_camera_direction_center">
+      <origin xyz="0.35 0 0" rpy="0 0 0"/>
+      <geometry>
+        <box size="0.7 0.018 0.018"/>
+      </geometry>
+      <material name="camera_direction_material"/>
+    </visual>
+    <visual name="back_camera_direction_left">
+      <origin xyz="0.267 0.225 0" rpy="0 0 0.6981"/>
+      <geometry>
+        <box size="0.7 0.014 0.014"/>
+      </geometry>
+      <material name="camera_direction_material"/>
+    </visual>
+    <visual name="back_camera_direction_right">
+      <origin xyz="0.267 -0.225 0" rpy="0 0 -0.6981"/>
+      <geometry>
+        <box size="0.7 0.014 0.014"/>
+      </geometry>
+      <material name="camera_direction_material"/>
+    </visual>
+    <visual name="back_camera_direction_top">
+      <origin xyz="0.296 0 0.187" rpy="0 -0.561 0"/>
+      <geometry>
+        <box size="0.7 0.014 0.014"/>
+      </geometry>
+      <material name="camera_direction_material"/>
+    </visual>
+    <visual name="back_camera_direction_bottom">
+      <origin xyz="0.296 0 -0.187" rpy="0 0.561 0"/>
+      <geometry>
+        <box size="0.7 0.014 0.014"/>
+      </geometry>
+      <material name="camera_direction_material"/>
+    </visual>
+    <visual name="back_camera_direction_tip">
+      <origin xyz="0.7 0 0" rpy="0 0 0"/>
+      <geometry>
+        <sphere radius="0.025"/>
+      </geometry>
+      <material name="camera_direction_material"/>
+    </visual>
+  </link>
+  <joint name="back_camera_rotated_joint" type="fixed">
+    <origin xyz="0 0 0" rpy="0 0 1.5708"/>
+    <parent link="back_camera_link"/>
+    <child link="back_camera_rotated_frame"/>
+  </joint>
   <!-- ============================================================ -->
   <!--  imu_link                                                    -->
